Commit message: Added EKF integration and stereo camera simulation

File: src/shrimp_modu/urdf/shrimp.urdf (robot description, URDF)
Before this commit: robot SHRIM_MECHANICAL_BACKUP, 10 links, 9 joints
Links:
- added link camera_link; collision box size=0.08 0.16 0.05; visual box size=0.08 0.16 0.05
- added link left_camera_frame
- added link left_camera_optical_frame
- added link right_camera_frame
- added link right_camera_optical_frame
Joints:
- added joint base_footprint_to_camera_link: type fixed, parent base_footprint, child camera_link, origin xyz=0.02 0 0.30 rpy=0 0 0
- added joint camera_link_to_left_camera_frame: type fixed, parent camera_link, child left_camera_frame, origin xyz=0 0.035 0 rpy=0 0 0
- added joint camera_link_to_right_camera_frame: type fixed, parent camera_link, child right_camera_frame, origin xyz=0 -0.035 0 rpy=0 0 0
- added joint left_camera_frame_to_left_camera_optical_frame: type fixed, parent left_camera_frame, child left_camera_optical_frame, origin xyz=0 0 0 rpy=-1.57079632679 0 -1.57079632679
- added joint right_camera_frame_to_right_camera_optical_frame: type fixed, parent right_camera_frame, child right_camera_optical_frame, origin xyz=0 0 0 rpy=-1.57079632679 0 -1.57079632679
